File: lineScope-5ASW-probe.kicad_pcb (KiCad board)
At the start: 2 copper layers, 99.5 x 30 mm, 23 parts, among them J1 Conn_01x03, T1 TA16-01

Commit message: Minor fixes
Parts:
- added REF**: WEEE-Logo_4.2x6mm_SilkScreen, Symbol:WEEE-Logo_4.2x6mm_SilkScreen, F.Cu at (181.5, 83.2)
- added REF**: Attention, Koszalix_Symbols:Attention, F.Cu at (102.2, 64.8)
- J1: value Conn_01x03 -> ~; footprint Connector_PinHeader_2.54mm:PinHeader_1x03_P2.54mm_Horizontal -> Koszalix_Connectors_Tab:TE-1-726388-2
- J4: value ~ -> Conn_01x03; footprint Koszalix_Connectors_Tab:TE-1-726388-2 -> Connector_PinHeader_2.54mm:PinHeader_1x03_P2.54mm_Horizontal
- moved J4 110.7 mm to (191.9, 70.1)
- moved J1 54.4 mm to (113.5, 79.0)
- moved J2 49.6 mm to (113.5, 66.2)
- moved DZ1 39.6 mm to (172.8, 70.1)
- moved DZ2 39.6 mm to (172.8, 75.1)
- moved FH1 39.6 mm to (120.2, 79.0)
- moved H2 39.6 mm to (191.6, 82.6)
- moved R2 39.6 mm to (168.6, 70.1)
- moved R4 39.6 mm to (168.6, 75.1)
- moved R5 39.6 mm to (186.7, 82.6)
- moved RV1 39.6 mm to (166.8, 70.1)
- moved RV2 39.6 mm to (166.8, 75.1)
- moved H3 39.6 mm to (191.6, 62.6)
- moved R6 39.6 mm to (186.7, 62.6)
- moved REF** 39.6 mm to (142.6, 60.6)
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Connections:
- J1 pad 1: Net-(J1-Pin_1) -> /HV.IN
- J2 pad 1: /HV.IN -> /HV.OUT
- J3 pad 1: /HV.OUT -> /HV.IN
- J4 pad 1: /HV.IN -> Net-(J4-Pin_1)
- R1 pad 2: Net-(J1-Pin_1) -> Net-(J4-Pin_1)
- R3 pad 2: Net-(J1-Pin_3) -> Net-(J4-Pin_3)
- R5 pad 2: unconnected-(R5-Pad2) -> GND
- R6 pad 2: unconnected-(R6-Pad2) -> GND
Routing:
- net Net-(J4-Pin_3): track 0.00 -> 5.15 mm
- net Net-(J4-Pin_1): track 0.00 -> 5.15 mm
- net Net-(J1-Pin_3): track 5.15 -> 0.00 mm
- net Net-(J1-Pin_1): track 5.15 -> 0.00 mm
Other:
- board text added: "0"
- board text added: "0 mm"
- board text added: "0,0000 mm / 0,0000 mm"
- board text added: "0,01 mm"
- board text added: "0,02"
- board text added: "0,035 mm"
- board text added: "0,3000 mm"
- board text added: "1"
- board text added: "1,51 mm"
- board text added: "1,6000 mm"
- board text added: "2"
- board text added: "3,3"
- board text added: "4,5"
- board text added: "99,5000 mm x 30,0000 mm"
- board text added: "B.Cu"
- board text added: "B.Mask"
- board text added: "B.Paste"
- board text added: "B.Silkscreen"
- board text added: "BOARD CHARACTERISTICS"
- board text added: "Board Thickness:"
- board text added: "Board overall dimensions:"
- board text added: "Bottom Silk Screen"
- board text added: "Bottom Solder Mask"
- board text added: "Bottom Solder Paste"
- board text added: "Castellated pads:"
- board text added: "Color"
- board text added: "Copper Finish:"
- board text added: "Copper Layer Count:"
- board text added: "Dielectric"
- board text added: "Edge card connectors:"
- board text added: "Epsilon R"
- board text added: "F.Cu"
- board text added: "F.Mask"
- board text added: "F.Paste"
- board text added: "F.Silkscreen"
- board text added: "FR4"
- board text added: "HIGH VOLTAGE"
- board text added: "Impedance Control:"
- board text added: "Layer Name"
- board text added: "Loss Tangent"
- board text added: "Material"
- board text added: "Min hole diameter:"
- board text added: "Min track/spacing:"
- board text added: "No"
- board text added: "None"
- board text added: "Not specified"
- board text added: "OUT+ GND OUT-"
- board text added: "Plated Board Edge:"
- board text added: "Thickness (mm)"
- board text added: "Top Silk Screen"
- board text added: "Top Solder Mask"
- board text added: "Top Solder Paste"
- board text added: "Type"
- board text added: "copper"
- board text added: "core"
