File: lineScope-5ASW-probe.kicad_pcb (KiCad board)
At the start: 2 copper layers, 99.5 x 30 mm, 25 parts, among them J4 Conn_01x03, T1 TA16-01

Commit message: Minor update
Connections:
- net /HV.IN renamed /HV_{LIN}
- net /HV.IN' renamed /HV_{L1}
- net /HV.OUT renamed /HV_{LOUT}
- net Net-(J4-Pin_1) renamed /OUT_{H}
- net Net-(J4-Pin_3) renamed /OUT_{L}
Changed lines of the file:
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@@
 	(net 6 "Net-(H2-Pad1)")
 	(net 7 "Net-(H3-Pad1)")
-	(net 8 "Net-(J4-Pin_3)")
-	(net 9 "Net-(J4-Pin_1)")
-	(net 10 "/HV.IN")
-	(net 11 "/HV.IN'")
-	(net 12 "/HV.OUT")
+	(net 8 "/HV_{L1}")
+	(net 9 "/HV_{LIN}")
+	(net 10 "/HV_{LOUT}")
+	(net 11 "/OUT_{H}")
+	(net 12 "/OUT_{L}")
 	(footprint "Resistor_SMD:R_0603_1608Metric"
 		(layer "F.Cu")
@@
 			(layers "*.Cu" "*.Mask")
 			(remove_unused_layers no)
-			(net 10 "/HV.IN")
+			(net 9 "/HV_{LIN}")
 			(pintype "passive")
 		)
@@
 			(layers "*.Cu" "*.Mask")
 			(remove_unused_layers no)
-			(net 10 "/HV.IN")
+			(net 9 "/HV_{LIN}")
 			(pintype "passive")
 		)
@@
 			(layers "*.Cu" "*.Mask")
 			(remove_unused_layers no)
-			(net 10 "/HV.IN")
+			(net 9 "/HV_{LIN}")
 			(pintype "passive")
 		)
@@
 			(layers "*.Cu" "*.Mask")
 			(remove_unused_layers no)
-			(net 11 "/HV.IN'")
+			(net 8 "/HV_{L1}")
 			(pintype "passive")
 		)
@@
 			(layers "F.Cu" "F.Paste" "F.Mask")
 			(roundrect_rratio 0.192308)
-			(net 8 "Net-(J4-Pin_3)")
+			(net 12 "/OUT_{L}")
 			(pintype "passive")
 		)
@@
 			(layers "*.Cu" "*.Mask")
 			(remove_unused_layers no)
-			(net 10 "/HV.IN")
+			(net 9 "/HV_{LIN}")
 			(pintype "passive")
 		)
@@
 			(layers "*.Cu" "*.Mask")
 			(remove_unused_layers no)
-			(net 10 "/HV.IN")
+			(net 9 "/HV_{LIN}")
 			(pintype "passive")
 		)
@@
 			(layers "*.Cu" "*.Mask")
 			(remove_unused_layers no)
-			(net 11 "/HV.IN'")
+			(net 8 "/HV_{L1}")
 			(pintype "passive")
 		)
@@
 			(layers "*.Cu" "*.Mask")
 			(remove_unused_layers no)
-			(net 12 "/HV.OUT")
+			(net 10 "/HV_{LOUT}")
 			(pintype "passive")
 		)
@@
 			(layers "F.Cu" "F.Paste" "F.Mask")
 			(roundrect_rratio 0.192308)
-			(net 9 "Net-(J4-Pin_1)")
+			(net 11 "/OUT_{H}")
 			(pintype "passive")
 		)
@@
 			(layers "*.Cu" "*.Mask")
 			(remove_unused_layers no)
-			(net 9 "Net-(J4-Pin_1)")
+			(net 11 "/OUT_{H}")
 			(pinfunction "Pin_1")
 			(pintype "passive")
@@
 			(layers "*.Cu" "*.Mask")
 			(remove_unused_layers no)
-			(net 8 "Net-(J4-Pin_3)")
+			(net 12 "/OUT_{L}")
 			(pinfunction "Pin_3")
 			(pintype "passive")
@@
 			(layers "*.Cu" "*.Mask")
 			(remove_unused_layers no)
-			(net 12 "/HV.OUT")
+			(net 10 "/HV_{LOUT}")
 			(pintype "passive")
 		)
@@
 			(layers "*.Cu" "*.Mask")
 			(remove_unused_layers no)
-			(net 12 "/HV.OUT")
+			(net 10 "/HV_{LOUT}")
 			(pintype "passive")
 		)
@@
 	)
 	(segment
-		(start 186.9625 75.1)
-		(end 192.1125 75.1)
-		(width 0.2)
+		(start 150.3825 79)
+		(end 150.4325 78.95)
+		(width 2)
 		(layer "F.Cu")
 		(net 8)
 	)
 	(segment
-		(start 192.1125 70.1)
-		(end 186.9625 70.1)
-		(width 0.2)
+		(start 142.8125 79)
+		(end 150.3825 79)
+		(width 2)
 		(layer "F.Cu")
-		(net 9)
+		(net 8)
 	)
 	(segment
@@
 		(width 2)
 		(layer "F.Cu")
-		(net 10)
+		(net 9)
 	)
 	(segment
@@
 		(width 2)
 		(layer "F.Cu")
-		(net 10)
+		(net 9)
 	)
 	(segment
@@
 		(width 2)
 		(layer "F.Cu")
-		(net 10)
+		(net 9)
 	)
 	(segment
@@
 		(width 2)
 		(layer "F.Cu")
-		(net 10)
+		(net 9)
 	)
 	(segment
@@
 		(width 2)
 		(layer "F.Cu")
-		(net 10)
+		(net 9)
 	)
 	(segment
-		(start 150.3825 79)
-		(end 150.4325 78.95)
+		(start 111.0225 66.25)
+		(end 110.9725 66.2)
 		(width 2)
 		(layer "F.Cu")
-		(net 11)
+		(net 10)
 	)
 	(segment
-		(start 142.8125 79)
-		(end 150.3825 79)
+		(start 150.4325 66.25)
+		(end 111.0225 66.25)
 		(width 2)
 		(layer "F.Cu")
-		(net 11)
+		(net 10)
 	)
 	(segment
-		(start 111.0225 66.25)
-		(end 110.9725 66.2)
-		(width 2)
+		(start 192.1125 70.1)
+		(end 186.9625 70.1)
+		(width 0.2)
 		(layer "F.Cu")
-		(net 12)
+		(net 11)
 	)
 	(segment
-		(start 150.4325 66.25)
-		(end 111.0225 66.25)
-		(width 2)
+		(start 186.9625 75.1)
+		(end 192.1125 75.1)
+		(width 0.2)
 		(layer "F.Cu")
 		(net 12)

Commit message: Change R2 to 100Ohm
Parts:
- R2: value 300R -> 100R
Changed lines of the file:
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@@
 			)
 		)
-		(property "Value" "300R"
+		(property "Value" "100R"
 			(at 0 1.43 -90)
 			(layer "F.Fab")
@@
 			)
 		)
-		(property "MPN" "RC0603FR-07300R"
+		(property "MPN" "RC0603FR-07100R"
 			(at 0 0 -90)
 			(unlocked yes)

Commit message: Bump revsion to 1.1.0
Other:
- board text added: "Rev 1.1.0 03/2024"
- board text removed: "Rev 1.0.0 03/2024"
Changed lines of the file:
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@@
 	(title_block
 		(title "lineScope 5A Probe")
-		(date "2024-03-21")
-		(rev "1.0.0")
+		(date "2024-05-26")
+		(rev "1.1.0")
 		(company "Koszalix")
 	)
@@
 		)
 	)
-	(gr_text "Rev 1.0.0 03/2024"
+	(gr_text "Rev 1.1.0 03/2024"
 		(at 116.6125 63.2 0)
 		(layer "F.SilkS")
