File: lineScope-5ASW-probe.kicad_sch (KiCad schematic)
At the start: 22 parts, among them J1 Conn_01x03, T1 TA16-01

Commit message: Minor fixes
Parts:
- added FF1: 500m/ FF, symbol Koszalix_Fuses:Fuse_5A_5x20_Ceramic_SuperFast
- renumbered J2 to J1, J3 to J2, J4 to J3, J1 to J4
Connections:
- net GND: now also R5.2, R6.2
- no-connect marks 0 -> 2
Other:
- company: (none) -> Koszalix
- title: (none) -> lineScope 5A Probe
Changed lines of the file:
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@@
 	(generator_version "8.0")
 	(paper "A4")
+	(title_block
+		(title "lineScope 5A Probe")
+		(date "2024-03-21")
+		(rev "1.0.0")
+		(company "Koszalix")
+	)
 	(junction
 		(at 155.575 88.9)
@@
 		(diameter 0)
 		(color 0 0 0 0)
+	)
+	(no_connect
+		(at 79.375 187.325)
+	)
+	(no_connect
+		(at 74.295 187.325)
 	)
 	(wire
@@
 		(on_board yes)
 		(dnp no)
-		(property "Reference" "J2"
+		(property "Reference" "J1"
 			(at 82.55 87.376 0)
 			(effects
@@
 			(project "lineScope-5ASW-probe"
 				(path "/32a3c3e3-fb97-4b0b-b0b8-7565b5e62235"
-					(reference "J2")
+					(reference "J1")
 					(unit 1)
 				)
@@
 		(on_board yes)
 		(dnp no)
-		(property "Reference" "J3"
+		(property "Reference" "J2"
 			(at 82.55 99.06 0)
 			(effects
@@
 			(project "lineScope-5ASW-probe"
 				(path "/32a3c3e3-fb97-4b0b-b0b8-7565b5e62235"
-					(reference "J3")
+					(reference "J2")
 					(unit 1)
 				)
@@
 			)
 		)
-		(property "Datasheet" ""
+		(property "Datasheet" "https://cdn.shopifycdn.net/s/files/1/2723/6858/files/TA16_cd4c8c8e-3e86-4eb8-806b-403a81fbd9c5.pdf?v=1632720467"
 			(at 114.935 88.9 0)
 			(effects
@@
 		(on_board yes)
 		(dnp no)
-		(property "Reference" "J4"
+		(property "Reference" "J3"
 			(at 82.55 91.186 0)
 			(effects
@@
 			(project "lineScope-5ASW-probe"
 				(path "/32a3c3e3-fb97-4b0b-b0b8-7565b5e62235"
-					(reference "J4")
+					(reference "J3")
 					(unit 1)
 				)
@@
 	)
 	(symbol
+		(lib_id "Koszalix_Fuses:Fuse_5A_5x20_Ceramic_SuperFast")
+		(at 74.295 187.325 0)
+		(unit 1)
+		(exclude_from_sim yes)
+		(in_bom yes)
+		(on_board no)
+		(dnp no)
+		(fields_autoplaced yes)
+		(property "Reference" "FF1"
+			(at 76.835 181.61 0)
+			(effects
+				(font
+					(size 1.27 1.27)
+				)
+			)
+		)
+		(property "Value" "500m/ FF"
+			(at 76.835 184.15 0)
+			(effects
+				(font
+					(size 1.27 1.27)
+				)
+			)
+		)
+		(property "Footprint" ""
+			(at 85.725 187.833 0)
+			(effects
+				(font
+					(size 1.27 1.27)
+				)
+				(justify left bottom)
+				(hide yes)
+			)
+		)
+		(property "Datasheet" "https://www.tme.eu/Document/614276a4b092aa9a63706d3ca24fbdad/SIBA-GSS-7000140.pdf"
+			(at 85.725 187.833 0)
+			(effects
+				(font
+					(size 1.27 1.27)
+				)
+				(justify left bottom)
+				(hide yes)
+			)
+		)
+		(property "Description" ""
+			(at 85.725 187.833 0)
+			(effects
+				(font
+					(size 1.27 1.27)
+				)
+				(justify left bottom)
+				(hide yes)
+			)
+		)
+		(property "MPN" "7000140.5"
+			(at 74.295 187.325 0)
+			(effects
+				(font
+					(size 1.27 1.27)
+				)
+				(hide yes)
+			)
+		)
+		(property "Manufacturer" "SIBA"
+			(at 74.295 187.325 0)
+			(effects
+				(font
+					(size 1.27 1.27)
+				)
+				(hide yes)
+			)
+		)
+		(pin "1"
+		)
+		(pin "2"
+		)
+		(instances
+			(project "lineScope-5ASW-probe"
+				(path "/32a3c3e3-fb97-4b0b-b0b8-7565b5e62235"
+					(reference "FF1")
+					(unit 1)
+				)
+			)
+		)
+	)
+	(symbol
+		(lib_id "power:GND")
+		(at 149.86 146.05 0)
+		(unit 1)
+		(exclude_from_sim no)
+		(in_bom yes)
+		(on_board yes)
+		(dnp no)
+		(fields_autoplaced yes)
+		(property "Reference" "#PWR07"
+			(at 149.86 152.4 0)
+			(effects
+				(font
+					(size 1.27 1.27)
+				)
+				(hide yes)
+			)
+		)
+		(property "Value" "GND"
+			(at 149.86 151.13 0)
+			(effects
+				(font
+					(size 1.27 1.27)
+				)
+			)
+		)
+		(property "Footprint" ""
+			(at 149.86 146.05 0)
+			(effects
+				(font
+					(size 1.27 1.27)
+				)
+				(hide yes)
+			)
+		)
+		(property "Datasheet" ""
+			(at 149.86 146.05 0)
+			(effects
+				(font
+					(size 1.27 1.27)
+				)
+				(hide yes)
+			)
+		)
+		(property "Description" "Power symbol creates a global label with name \"GND\" , ground"
+			(at 149.86 146.05 0)
+			(effects
+				(font
+					(size 1.27 1.27)
+				)
+				(hide yes)
+			)
+		)
+		(pin "1"
+		)
+		(instances
+			(project "lineScope-5ASW-probe"
+				(path "/32a3c3e3-fb97-4b0b-b0b8-7565b5e62235"
+					(reference "#PWR07")
+					(unit 1)
+				)
+			)
+		)
+	)
+	(symbol
 		(lib_id "Koszalix_Varistors:MCVZ0603M180AGT")
 		(at 146.05 111.125 0)
@@
 		(on_board yes)
 		(dnp no)
-		(property "Reference" "J1"
+		(property "Reference" "J4"
 			(at 198.12 93.3449 0)
 			(effects
@@
 			(project "lineScope-5ASW-probe"
 				(path "/32a3c3e3-fb97-4b0b-b0b8-7565b5e62235"
-					(reference "J1")
+					(reference "J4")
 					(unit 1)
 				)
@@
 					(unit 1)
 				)
+			)
+		)
+	)
+	(symbol
+		(lib_id "power:GND")
+		(at 173.99 145.415 0)
+		(unit 1)
+		(exclude_from_sim no)
+		(in_bom yes)
+		(on_board yes)
+		(dnp no)
+		(fields_autoplaced yes)
+		(property "Reference" "#PWR08"
+			(at 173.99 151.765 0)
+			(effects
+				(font
+					(size 1.27 1.27)
+				)
+				(hide yes)
+			)
+		)
+		(property "Value" "GND"
+			(at 173.99 150.495 0)
+			(effects
+				(font
+					(size 1.27 1.27)
+				)
+			)
+		)
+		(property "Footprint" ""
+			(at 173.99 145.415 0)
+			(effects
+				(font
+					(size 1.27 1.27)
+				)
+				(hide yes)
+			)
+		)
+		(property "Datasheet" ""
+			(at 173.99 145.415 0)
+			(effects
+				(font
+					(size 1.27 1.27)
+				)
+				(hide yes)
+			)
+		)
+		(property "Description" "Power symbol creates a global label with name \"GND\" , ground"
+			(at 173.99 145.415 0)
+			(effects
+				(font
+					(size 1.27 1.27)
+				)
+				(hide yes)
+			)
+		)
+		(pin "1"
+		)
+		(instances
+			(project "lineScope-5ASW-probe"
+				(path "/32a3c3e3-fb97-4b0b-b0b8-7565b5e62235"
+					(reference "#PWR08")
+					(unit 1)
+				)
