File: lineScope-5ASW-probe.kicad_sch (KiCad schematic)
At the start: 23 parts, among them J4 Conn_01x03, T1 TA16-01

Commit message: Minor update
Connections:
- net OUT_{H}: now reaches J4.1 (Pin_1), R1.2
- net OUT_{L}: now reaches J4.3 (Pin_3), R3.2
- net HV.IN renamed HV_{LIN}
- net HV.IN' renamed HV_{L1}
- net HV.OUT renamed HV_{LOUT}
Other:
- moved on the sheet: R1, R3
Changed lines of the file:
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@@
 	(wire
 		(pts
-			(xy 183.515 100.33) (xy 186.055 100.33)
+			(xy 180.975 100.33) (xy 186.055 100.33)
 		)
 		(stroke
@@
 	(wire
 		(pts
-			(xy 175.895 88.9) (xy 155.575 88.9)
+			(xy 173.355 88.9) (xy 155.575 88.9)
 		)
 		(stroke
@@
 	(wire
 		(pts
-			(xy 186.055 88.9) (xy 183.515 88.9)
+			(xy 186.055 88.9) (xy 180.975 88.9)
 		)
 		(stroke
@@
 	(wire
 		(pts
-			(xy 165.1 100.33) (xy 175.895 100.33)
+			(xy 165.1 100.33) (xy 173.355 100.33)
 		)
 		(stroke
@@
 		)
 	)
-	(label "HV.OUT"
+	(label "HV_{LOUT}"
 		(at 92.075 100.33 0)
 		(fields_autoplaced yes)
@@
 		)
 	)
-	(label "HV.IN"
-		(at 92.075 88.9 0)
+	(label "OUT_{H}"
+		(at 186.055 88.9 180)
 		(fields_autoplaced yes)
 		(effects
@@
 				(size 1.27 1.27)
 			)
-			(justify left bottom)
-		)
-	)
-	(label "HV.IN'"
-		(at 107.95 88.9 0)
+			(justify right bottom)
+		)
+	)
+	(label "HV_{LIN}"
+		(at 92.075 88.9 0)
 		(fields_autoplaced yes)
 		(effects
@@
 		)
 	)
+	(label "HV_{L1}"
+		(at 107.95 88.9 0)
+		(fields_autoplaced yes)
+		(effects
+			(font
+				(size 1.27 1.27)
+			)
+			(justify left bottom)
+		)
+	)
+	(label "OUT_{L}"
+		(at 186.055 100.33 180)
+		(fields_autoplaced yes)
+		(effects
+			(font
+				(size 1.27 1.27)
+			)
+			(justify right bottom)
+		)
+	)
 	(symbol
 		(lib_id "Mechanical:MountingHole")
@@
 	(symbol
 		(lib_id "Device:R")
-		(at 179.705 100.33 90)
+		(at 177.165 100.33 90)
 		(unit 1)
 		(exclude_from_sim no)
@@
 		(fields_autoplaced yes)
 		(property "Reference" "R3"
-			(at 179.705 93.98 90)
+			(at 177.165 93.98 90)
 			(effects
 				(font
@@
 		)
 		(property "Value" "0R"
-			(at 179.705 96.52 90)
+			(at 177.165 96.52 90)
 			(effects
 				(font
@@
 		)
 		(property "Footprint" "Resistor_SMD:R_1206_3216Metric_Pad1.30x1.75mm_HandSolder"
-			(at 179.705 102.108 90)
+			(at 177.165 102.108 90)
 			(effects
 				(font
@@
 		)
 		(property "Datasheet" "~"
-			(at 179.705 100.33 0)
+			(at 177.165 100.33 0)
 			(effects
 				(font
@@
 		)
 		(property "Description" "Resistor"
-			(at 179.705 100.33 0)
+			(at 177.165 100.33 0)
 			(effects
 				(font
@@
 	(symbol
 		(lib_id "Device:R")
-		(at 179.705 88.9 90)
+		(at 177.165 88.9 90)
 		(unit 1)
 		(exclude_from_sim no)
@@
 		(fields_autoplaced yes)
 		(property "Reference" "R1"
-			(at 179.705 82.55 90)
+			(at 177.165 82.55 90)
 			(effects
 				(font
@@
 		)
 		(property "Value" "0R"
-			(at 179.705 85.09 90)
+			(at 177.165 85.09 90)
 			(effects
 				(font
@@
 		)
 		(property "Footprint" "Resistor_SMD:R_1206_3216Metric_Pad1.30x1.75mm_HandSolder"
-			(at 179.705 90.678 90)
+			(at 177.165 90.678 90)
 			(effects
 				(font
@@
 		)
 		(property "Datasheet" "~"
-			(at 179.705 88.9 0)
+			(at 177.165 88.9 0)
 			(effects
 				(font
@@
 		)
 		(property "Description" "Resistor"
-			(at 179.705 88.9 0)
-			(effects
-				(font
+			(at 177.165 88.9 0)
+			(effects
+				(font

Commit message: Change R2 to 100Ohm
Parts:
- removed R2: 300R, Resistor_SMD:R_0603_1608Metric, symbol Koszalix_Resistors_Yageo_RC0603:RES_300R_0603
- added R2: 100R, Resistor_SMD:R_0603_1608Metric, symbol Koszalix_Resistors_Yageo_RC0603:RES_100R_0603
Connections:
- net at DZ1.1, R1.1, RV1.1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: now also R2.1
- net at DZ2.1, R3.1, R4.1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: now also R2.2
